File: AergoPcb.kicad_pcb (KiCad board)
At the start: 2 copper layers, 159.6 x 139.8 mm, 239 parts, among them J1 Conn_01x15, J2 Conn_01x15, J3 Conn_01x04, M1 Mosfet-DMN63D8L, SW1 SW_Push, U1 ATmega32U4-AU, Y1 16MHz

Commit message: Finalized PCB and created Gerbers
Parts:
- added G***: LOGO, Aces Footprints:AceDragon, F.Cu at (235.8, 187.9)
- added REF**: breakaway-mousebites, random-keyboard-parts:breakaway-mousebites, F.Cu at (222.1, 173.1)
- added REF**: breakaway-mousebites, random-keyboard-parts:breakaway-mousebites, F.Cu at (225.1, 173.1)
- added REF**: breakaway-mousebites, random-keyboard-parts:breakaway-mousebites, F.Cu at (221.4, 122.7)
- added REF**: breakaway-mousebites, random-keyboard-parts:breakaway-mousebites, F.Cu at (225.8, 122.6)
- added U2: PRTR5V0U2X, random-keyboard-parts:SOT143B, B.Cu at (198.6, 102.0)
- C1, C2, C3, C4, C5, C6, C7, F1, J3, M1, R1, R2, R3, R4, R78, SW1, U1, Y1: moved to B.Cu
- moved Y1 170.6 mm to (209.0, 195.3), turned to 45 degrees
- moved C6 166.6 mm to (214.0, 196.2), turned to 270 degrees
- moved M1 159.8 mm to (197.8, 195.4), turned to 270 degrees
- moved R78 159.0 mm to (195.2, 192.0), turned to 90 degrees
- moved C5 158.2 mm to (204.1, 196.2), turned to 270 degrees
- moved C4 157.5 mm to (218.9, 185.2)
- moved C3 157.4 mm to (200.7, 188.1), turned to 270 degrees
- moved C1 152.1 mm to (217.6, 188.2)
- moved U1 151.6 mm to (208.5, 181.4), turned to 180 degrees
- moved C7 147.5 mm to (219.2, 181.0)
- moved R2 145.0 mm to (218.7, 174.6), turned to 90 degrees
- moved R4 137.5 mm to (199.6, 173.4), turned to 270 degrees
- moved R1 136.7 mm to (216.8, 174.6), turned to 90 degrees
- moved C2 135.8 mm to (213.0, 173.0), turned to 180 degrees
- moved SW1 134.7 mm to (177.6, 156.2), turned to 180 degrees
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Connections:
- net Net-(R1-Pad1) renamed D-
- net Net-(R2-Pad1) renamed D+
- J1 pad 10: COl12 -> COL12
- MX_PGDN1 pad 1: Net-(MX_PGDN1-Pad1) -> COL6
- R311 pad 1: Net-(MXIL1-Pad4) -> Net-(MX_I1-Pad4)
- U1 pad 10: Net-(U1-Pad10) -> COL9
- U1 pad 11: Net-(U1-Pad11) -> COL8
- U1 pad 19: Net-(U1-Pad19) -> COL6
- U1 pad 20: Net-(U1-Pad20) -> SwLedPWM
- U1 pad 21: Net-(U1-Pad21) -> COL0
- U1 pad 22: Net-(U1-Pad22) -> ROW1
- U1 pad 25: Net-(U1-Pad25) -> ROW5
- U1 pad 26: Net-(U1-Pad26) -> COL1
- U1 pad 27: Net-(U1-Pad27) -> COL2
- U1 pad 28: Net-(U1-Pad28) -> COL3
- U1 pad 29: Net-(U1-Pad29) -> COL4
- U1 pad 30: Net-(U1-Pad30) -> ROW0
- U1 pad 31: Net-(U1-Pad31) -> COL5
- U1 pad 32: Net-(U1-Pad32) -> ROW4
- U1 pad 36: Net-(U1-Pad36) -> ROW3
- U1 pad 37: Net-(U1-Pad37) -> ROW2
- U1 pad 38: Net-(U1-Pad38) -> COL7
- U1 pad 39: Net-(U1-Pad39) -> COL13
- U1 pad 40: Net-(U1-Pad40) -> COL12
- U1 pad 41: Net-(U1-Pad41) -> COL11
- U1 pad 9: Net-(U1-Pad9) -> COL10
Routing:
- net +5V: track 0.00 -> 968.4 mm, vias 0 -> 14
- net LedGND: track 0.00 -> 907.5 mm
- net ROW1: track 0.00 -> 319.4 mm, vias 0 -> 6
- net ROW5: track 0.00 -> 280.5 mm, vias 0 -> 2
- net ROW4: track 0.00 -> 279.3 mm, vias 0 -> 2
- net ROW0: track 0.00 -> 270.1 mm, vias 0 -> 2
- net COL0: track 0.00 -> 256.3 mm, vias 0 -> 2
- net ROW3: track 0.00 -> 224.4 mm, vias 0 -> 3
- net COL1: track 0.00 -> 221.7 mm, vias 0 -> 1
- net ROW2: track 0.00 -> 218.2 mm, vias 0 -> 3
- net COL2: track 0.00 -> 202.7 mm, vias 0 -> 1
- net GND: track 0.00 -> 198.1 mm, vias 0 -> 2
- net COL3: track 0.00 -> 197.0 mm, vias 0 -> 1
- net COL4: track 0.00 -> 164.6 mm, vias 0 -> 1
- net COL5: track 0.00 -> 150.1 mm, vias 0 -> 1
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- added copper zone on B.Cu, net GND
Other:
- board size 159.6 x 139.8 mm -> 299.2 x 140.2 mm
- rule pad_to_mask_clearance: 0.051 -> 0.2
- board text added: "AErgo V1"
- board text added: "by AceRecon"

Commit message: remade gerbers
Other:
- board size 299.2 x 140.2 mm -> 299.2 x 140 mm
Changed lines of the file:
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@@
   (general
     (thickness 1.6)
-    (drawings 61)
+    (drawings 60)
     (tracks 2344)
     (zones 0)
@@
       (net 2 GND))
   )
-  (dimension 120.2944 (width 0.3) (layer F.SilkS)
-    (gr_text "120.294 mm" (at 374.464 121.793 90) (layer F.SilkS)
-      (effects (font (size 1.5 1.5) (thickness 0.3)))
-    )
-    (feature1 (pts (xy 372.364 61.6458) (xy 372.950421 61.6458)))
-    (feature2 (pts (xy 372.364 181.9402) (xy 372.950421 181.9402)))
-    (crossbar (pts (xy 372.364 181.9402) (xy 372.364 61.6458)))
-    (arrow1a (pts (xy 372.364 61.6458) (xy 372.950421 62.772304)))
-    (arrow1b (pts (xy 372.364 61.6458) (xy 371.777579 62.772304)))
-    (arrow2a (pts (xy 372.364 181.9402) (xy 372.950421 180.813696)))
-    (arrow2b (pts (xy 372.364 181.9402) (xy 371.777579 180.813696)))
-  )
-  (dimension 299.365956 (width 0.3) (layer F.SilkS)
-    (gr_text "299.366 mm" (at 223.462347 64.329988 359.8152696) (layer F.SilkS)
-      (effects (font (size 1.5 1.5) (thickness 0.3)))
-    )
-    (feature1 (pts (xy 373.1514 62.6872) (xy 373.149427 63.299017)))
-    (feature2 (pts (xy 73.787 61.722) (xy 73.785027 62.333817)))
-    (crossbar (pts (xy 73.786918 61.747399) (xy 373.151318 62.712599)))
-    (arrow1a (pts (xy 373.151318 62.712599) (xy 372.022929 63.295385)))
-    (arrow1b (pts (xy 373.151318 62.712599) (xy 372.026711 62.122549)))
-    (arrow2a (pts (xy 73.786918 61.747399) (xy 74.911525 62.337449)))
-    (arrow2b (pts (xy 73.786918 61.747399) (xy 74.915307 61.164613)))
-  )
+  (gr_line (start 73.914 62.3062) (end 73.914 86.614) (layer Edge.Cuts) (width 0.15))
+  (gr_arc (start 74.4982 62.3062) (end 74.4982 61.722) (angle -90) (layer Edge.Cuts) (width 0.15))
+  (gr_line (start 99.568 61.722) (end 74.4982 61.722) (layer Edge.Cuts) (width 0.15))
   (gr_text "by AceRecon\n" (at 234.0356 172.6946) (layer F.SilkS)
     (effects (font (size 1.5 1.5) (thickness 0.3)))
@@
   (gr_line (start 118.618 61.722) (end 139.7 63.5) (layer Edge.Cuts) (width 0.15))
   (gr_line (start 99.568 61.722) (end 118.618 61.722) (layer Edge.Cuts) (width 0.15))
-  (gr_line (start 73.914 61.468) (end 99.568 61.722) (layer Edge.Cuts) (width 0.15))
-  (gr_line (start 73.914 86.614) (end 73.914 61.468) (layer Edge.Cuts) (width 0.15))
   (gr_line (start 73.914 180.848) (end 73.914 86.614) (layer Edge.Cuts) (width 0.15))
   (gr_arc (start 74.676 180.848) (end 73.914 180.848) (angle -90) (layer Edge.Cuts) (width 0.15))

Commit message: more pcb work
Parts:
- R11, R110, R111, R112, R113, R114, R12, R13, R14, R15, R16, R19, R21, R210, R211, R212, R213, R214, R22, R23, R24, R25, R26, R27, R28, R29, R31, R310, R311, R312, R313, R314, R32, R33, R34, R35, R36, R37, R38, R39, R41, R410, R411, R412, R413, R414, R42, R43, R44, R45, R46, R47, R48, R49, R51, R510, R511, R512, R513, R514, R52, R53, R54, R55, R56, R59, R61, R610, R611, R614, R64, R66, R69: value 800 -> 1k
