File: matrix.sch (KiCad schematic (older format))
At the start: 222 parts, among them J1 Conn_01x15, J2 Conn_01x15

Commit message: added jst footprints, continued work on pcb
Parts:
- removed J1, J2: Conn_01x15, symbol Connector_Generic:Conn_01x15
- added J? (x2): Conn_01x07, symbol Connector_Generic:Conn_01x07
- added J? (x2): Conn_01x08, symbol Connector_Generic:Conn_01x08
- added M1: Mosfet-DMN63D8L, symbol Ace's~Schematic~Symbols:Mosfet-DMN63D8L
- D1, D10, D11, D12, D13, D14, D15, D16, D17, D18, D19, D2, D20, D21, D22, D23, D24, D25, D26, D27, D28, D29, D3, D30, D31, D32, D33, D34, D35, D36, D37, D38, D39, D4, D40, D41, D42, D43, D44, D45, D46, D47, D48, D49, D5, D50, D51, D52, D53, D54, D55, D56, D57, D58, D59, D6, D60, D61, D62, D63, D64, D65, D66, D67, D68, D69, D7, D70, D71, D72, D73, D8, D9: footprint (none) -> Diode_SMD:D_SOD-123
- MX1, MX10, MX11, MX12, MX13, MX14, MX15, MX16, MX18, MX19, MX2, MX20, MX21, MX22, MX23, MX24, MX25, MX26, MX27, MX29, MX3, MX30, MX31, MX32, MX33, MX34, MX35, MX36, MX37, MX38, MX39, MX4, MX40, MX41, MX42, MX43, MX44, MX46, MX47, MX48, MX49, MX5, MX50, MX52, MX53, MX54, MX55, MX56, MX57, MX58, MX59, MX60, MX61, MX62, MX63, MX64, MX65, MX66, MX67, MX68, MX69, MX7, MX70, MX71, MX72, MX8, MX9: footprint (none) -> MX_Alps_Hybrid:MX-1U
- MX17, MX6, MX73: footprint (none) -> MX_Alps_Hybrid:MX-1.5U
- MX28: footprint (none) -> MX_Alps_Hybrid:MX-2.75U-FLIPPED
- MX45: footprint (none) -> MX_Alps_Hybrid:MX-1.25U
- MX51: footprint (none) -> MX_Alps_Hybrid:MX-2U-FLIPPED
- R10, R11, R12, R13, R14, R15, R16, R17, R18, R19, R20, R21, R22, R23, R24, R25, R26, R27, R28, R29, R30, R31, R32, R33, R34, R35, R36, R37, R38, R39, R40, R41, R42, R43, R44, R45, R46, R47, R48, R49, R5, R50, R51, R52, R53, R54, R55, R56, R57, R58, R59, R6, R60, R61, R62, R63, R64, R65, R66, R67, R68, R69, R7, R70, R71, R72, R73, R74, R75, R76, R77, R8, R9: footprint (none) -> Resistor_SMD:R_0805_2012Metric
- R78: renamed from R?; footprint (none) -> Resistor_SMD:R_0805_2012Metric
Other:
- moved on the sheet: R78

Commit message: finished right half, loaded keyboard parts pretty
Parts:
- removed J? (x2): Conn_01x07, symbol Connector_Generic:Conn_01x07
- removed J? (x2): Conn_01x08, symbol Connector_Generic:Conn_01x08
- added J1, J2: Conn_01x15, Connector_JST:JST_SH_SM15B-SRSS-TB_1x15-1MP_P1.00mm_Horizontal, symbol Connector_Generic:Conn_01x15
- M1: footprint (none) -> Ace's Footprints:Mosfet-DMN63D8L
- MXIL1: renamed from MX54; footprint MX_Alps_Hybrid:MX-1U -> MX_Alps_Hybrid:MXOnly-1U
- MX_'1: renamed from MX71; value MX-1U -> MX-1.25U; footprint MX_Alps_Hybrid:MX-1U -> MX_Alps_Hybrid:MXOnly-1.25U
- MX_-1: renamed from MX59; footprint MX_Alps_Hybrid:MX-1U -> MX_Alps_Hybrid:MXOnly-1U
- MX_/1: renamed from MX67; footprint MX_Alps_Hybrid:MX-1U -> MX_Alps_Hybrid:MXOnly-1U
- MX_0: renamed from MX53; footprint MX_Alps_Hybrid:MX-1U -> MX_Alps_Hybrid:MXOnly-1U
- MX_1: renamed from MX8; footprint MX_Alps_Hybrid:MX-1U -> MX_Alps_Hybrid:MXOnly-1U
- MX_2: renamed from MX13; footprint MX_Alps_Hybrid:MX-1U -> MX_Alps_Hybrid:MXOnly-1U
- MX_3: renamed from MX19; footprint MX_Alps_Hybrid:MX-1U -> MX_Alps_Hybrid:MXOnly-1U
- MX_4: renamed from MX24; footprint MX_Alps_Hybrid:MX-1U -> MX_Alps_Hybrid:MXOnly-1U
- MX_5: renamed from MX30; footprint MX_Alps_Hybrid:MX-1U -> MX_Alps_Hybrid:MXOnly-1U
- MX_6: renamed from MX34; footprint MX_Alps_Hybrid:MX-1U -> MX_Alps_Hybrid:MXOnly-1U
- MX_7: renamed from MX37; footprint MX_Alps_Hybrid:MX-1U -> MX_Alps_Hybrid:MXOnly-1U
- MX_8: renamed from MX41; footprint MX_Alps_Hybrid:MX-1U -> MX_Alps_Hybrid:MXOnly-1U
- MX_9: renamed from MX47; footprint MX_Alps_Hybrid:MX-1U -> MX_Alps_Hybrid:MXOnly-1U
- MX_;1: renamed from MX66; footprint MX_Alps_Hybrid:MX-1U -> MX_Alps_Hybrid:MXOnly-1U
- MX_<1: renamed from MX56; footprint MX_Alps_Hybrid:MX-1U -> MX_Alps_Hybrid:MXOnly-1U
- MX_=1: renamed from MX64; footprint MX_Alps_Hybrid:MX-1U -> MX_Alps_Hybrid:MXOnly-1U
- MX_>1: renamed from MX62; footprint MX_Alps_Hybrid:MX-1U -> MX_Alps_Hybrid:MXOnly-1U
- MX_A1: renamed from MX10; footprint MX_Alps_Hybrid:MX-1U -> MX_Alps_Hybrid:MXOnly-1U
- MX_B1: renamed from MX33; footprint MX_Alps_Hybrid:MX-1U -> MX_Alps_Hybrid:MXOnly-1U
- MX_BackSpace1: renamed from MX69; footprint MX_Alps_Hybrid:MX-1U -> MX_Alps_Hybrid:MXOnly-1U
- MX_C1: renamed from MX22; footprint MX_Alps_Hybrid:MX-1U -> MX_Alps_Hybrid:MXOnly-1U
- MX_D1: renamed from MX21; footprint MX_Alps_Hybrid:MX-1U -> MX_Alps_Hybrid:MXOnly-1U
- MX_DEL1: renamed from MX70; footprint MX_Alps_Hybrid:MX-1U -> MX_Alps_Hybrid:MXOnly-1U
- MX_E1: renamed from MX20; footprint MX_Alps_Hybrid:MX-1U -> MX_Alps_Hybrid:MXOnly-1U
- MX_END1: renamed from MX39; footprint MX_Alps_Hybrid:MX-1U -> MX_Alps_Hybrid:MXOnly-1U
- MX_ENTER1: renamed from MX51; value MX-2U-FLIPPED -> MX-2U; footprint MX_Alps_Hybrid:MX-2U-FLIPPED -> MX_Alps_Hybrid:MXOnly-2U-ReversedStabilizers; symbol MX_Alps_Hybrids:MX-2U-FLIPPED -> MX_Alps_Hybrids:MX-2U
- MX_ESC1: renamed from MX2; footprint MX_Alps_Hybrid:MX-1U -> MX_Alps_Hybrid:MXOnly-1U
- MX_F1: renamed from MX1; footprint MX_Alps_Hybrid:MX-1U -> MX_Alps_Hybrid:MXOnly-1U
- MX_F10: renamed from MX58; footprint MX_Alps_Hybrid:MX-1U -> MX_Alps_Hybrid:MXOnly-1U
- MX_F11: renamed from MX63; footprint MX_Alps_Hybrid:MX-1U -> MX_Alps_Hybrid:MXOnly-1U
- MX_F12: renamed from MX68; footprint MX_Alps_Hybrid:MX-1U -> MX_Alps_Hybrid:MXOnly-1U
- MX_F13: renamed from MX26; footprint MX_Alps_Hybrid:MX-1U -> MX_Alps_Hybrid:MXOnly-1U
- MX_F2: renamed from MX7; footprint MX_Alps_Hybrid:MX-1U -> MX_Alps_Hybrid:MXOnly-1U
- MX_F3: renamed from MX12; footprint MX_Alps_Hybrid:MX-1U -> MX_Alps_Hybrid:MXOnly-1U
- MX_F4: renamed from MX18; footprint MX_Alps_Hybrid:MX-1U -> MX_Alps_Hybrid:MXOnly-1U
- MX_F5: renamed from MX23; footprint MX_Alps_Hybrid:MX-1U -> MX_Alps_Hybrid:MXOnly-1U
- MX_F6: renamed from MX29; footprint MX_Alps_Hybrid:MX-1U -> MX_Alps_Hybrid:MXOnly-1U
- MX_F7: renamed from MX40; footprint MX_Alps_Hybrid:MX-1U -> MX_Alps_Hybrid:MXOnly-1U
- MX_F8: renamed from MX46; footprint MX_Alps_Hybrid:MX-1U -> MX_Alps_Hybrid:MXOnly-1U
- MX_F9: renamed from MX52; footprint MX_Alps_Hybrid:MX-1U -> MX_Alps_Hybrid:MXOnly-1U
- MX_FN1: renamed from MX6; footprint MX_Alps_Hybrid:MX-1.5U -> MX_Alps_Hybrid:MXOnly-1.5U
- MX_FN2: renamed from MX45; footprint MX_Alps_Hybrid:MX-1.25U -> MX_Alps_Hybrid:MXOnly-1.25U
- MX_G1: renamed from MX32; footprint MX_Alps_Hybrid:MX-1U -> MX_Alps_Hybrid:MXOnly-1U
- MX_H1: renamed from MX43; footprint MX_Alps_Hybrid:MX-1U -> MX_Alps_Hybrid:MXOnly-1U
- MX_HOME1: renamed from MX38; footprint MX_Alps_Hybrid:MX-1U -> MX_Alps_Hybrid:MXOnly-1U
- MX_J1: renamed from MX49; footprint MX_Alps_Hybrid:MX-1U -> MX_Alps_Hybrid:MXOnly-1U
- MX_K1: renamed from MX55; footprint MX_Alps_Hybrid:MX-1U -> MX_Alps_Hybrid:MXOnly-1U
- MX_L1: renamed from MX61; footprint MX_Alps_Hybrid:MX-1U -> MX_Alps_Hybrid:MXOnly-1U
- MX_LALT1: renamed from MX17; footprint MX_Alps_Hybrid:MX-1.5U -> MX_Alps_Hybrid:MXOnly-1.5U
- MX_LCTRL1: renamed from MX4; value MX-1U -> MX-1.25U; footprint MX_Alps_Hybrid:MX-1U -> MX_Alps_Hybrid:MXOnly-1.25U; symbol MX_Alps_Hybrids:MX-1U -> MX_Alps_Hybrids:MX-1.25U
- MX_LSHIFT1: renamed from MX5; value MX-1U -> MX-1.25U; footprint MX_Alps_Hybrid:MX-1U -> MX_Alps_Hybrid:MXOnly-1.25U; symbol MX_Alps_Hybrids:MX-1U -> MX_Alps_Hybrids:MX-1.25U
- MX_M1: renamed from MX50; footprint MX_Alps_Hybrid:MX-1U -> MX_Alps_Hybrid:MXOnly-1U
- MX_N1: renamed from MX44; footprint MX_Alps_Hybrid:MX-1U -> MX_Alps_Hybrid:MXOnly-1U
- MX_O1: renamed from MX60; footprint MX_Alps_Hybrid:MX-1U -> MX_Alps_Hybrid:MXOnly-1U
- MX_P1: renamed from MX65; footprint MX_Alps_Hybrid:MX-1U -> MX_Alps_Hybrid:MXOnly-1U
- MX_PGDN1: renamed from MX36; footprint MX_Alps_Hybrid:MX-1U -> MX_Alps_Hybrid:MXOnly-1U
- MX_PGUP1: renamed from MX35; footprint MX_Alps_Hybrid:MX-1U -> MX_Alps_Hybrid:MXOnly-1U
- MX_Q1: renamed from MX9; footprint MX_Alps_Hybrid:MX-1U -> MX_Alps_Hybrid:MXOnly-1U
- MX_R1: renamed from MX25; footprint MX_Alps_Hybrid:MX-1U -> MX_Alps_Hybrid:MXOnly-1U
- MX_RALT1: renamed from MX57; footprint MX_Alps_Hybrid:MX-1U -> MX_Alps_Hybrid:MXOnly-1U
- MX_RCTRL1: renamed from MX73; footprint MX_Alps_Hybrid:MX-1.5U -> MX_Alps_Hybrid:MXOnly-1.5U
- MX_RSHIFT1: renamed from MX72; value MX-1U -> MX-1.25U; footprint MX_Alps_Hybrid:MX-1U -> MX_Alps_Hybrid:MXOnly-1.25U; symbol MX_Alps_Hybrids:MX-1U -> MX_Alps_Hybrids:MX-1.25U
- MX_S1: renamed from MX15; footprint MX_Alps_Hybrid:MX-1U -> MX_Alps_Hybrid:MXOnly-1U
- MX_SPACE1: renamed from MX28; value MX-2.75U-FLIPPED -> MX-2.75U; footprint MX_Alps_Hybrid:MX-2.75U-FLIPPED -> MX_Alps_Hybrid:MXOnly-2.75U-ReversedStabilizers; symbol MX_Alps_Hybrids:MX-2.75U-FLIPPED -> MX_Alps_Hybrids:MX-2.75U
- MX_T1: renamed from MX31; footprint MX_Alps_Hybrid:MX-1U -> MX_Alps_Hybrid:MXOnly-1U
- MX_TAB1: renamed from MX3; footprint MX_Alps_Hybrid:MX-1U -> MX_Alps_Hybrid:MXOnly-1U
- MX_U1: renamed from MX48; footprint MX_Alps_Hybrid:MX-1U -> MX_Alps_Hybrid:MXOnly-1U
- MX_V1: renamed from MX27; footprint MX_Alps_Hybrid:MX-1U -> MX_Alps_Hybrid:MXOnly-1U
- MX_W1: renamed from MX14; footprint MX_Alps_Hybrid:MX-1U -> MX_Alps_Hybrid:MXOnly-1U
- MX_X1: renamed from MX16; footprint MX_Alps_Hybrid:MX-1U -> MX_Alps_Hybrid:MXOnly-1U
- MX_Y1: renamed from MX42; footprint MX_Alps_Hybrid:MX-1U -> MX_Alps_Hybrid:MXOnly-1U
- MX_Z1: renamed from MX11; footprint MX_Alps_Hybrid:MX-1U -> MX_Alps_Hybrid:MXOnly-1U
- renumbered D1 to D11, D46 to D110, D52 to D111, D58 to D112, D63 to D113, D68 to D114, D7 to D12, D12 to D13, D18 to D14, D23 to D15, D29 to D16, D40 to D19, D2 to D21, D47 to D210, D53 to D211, D59 to D212, D64 to D213, D69 to D214, D8 to D22, D13 to D23, D19 to D24, D24 to D25, D30 to D26, D34 to D27, D37 to D28, D41 to D29, D3 to D31, D48 to D310, D54 to D311, D60 to D312, D65 to D313, D70 to D314, D9 to D32, D14 to D33, D20 to D34, D25 to D35, D31 to D36, D35 to D37, D42 to D39, D4 to D41, D49 to D410, D55 to D411, D61 to D412, D66 to D413, D71 to D414, D10 to D42, D15 to D43, D21 to D44, D26 to D45, D32 to D46, D36 to D47, D39 to D48, D43 to D49, D5 to D51, D50 to D510, D56 to D511, D62 to D512, D67 to D513, D72 to D514, D11 to D52, D16 to D53, D22 to D54, D27 to D55, D33 to D56, D44 to D59, D6 to D61, D51 to D610, D57 to D611, D73 to D614, D17 to D64, D28 to D66, D45 to D69, R5 to R11, R50 to R110, R56 to R111, R62 to R112, R67 to R113, R72 to R114, R11 to R12, R16 to R13, R22 to R14, R27 to R15, R33 to R16, R44 to R19, R6 to R21, R51 to R210, R57 to R211, R63 to R212, R68 to R213, R73 to R214, R12 to R22, R17 to R23, R23 to R24, R28 to R25, R34 to R26, R38 to R27, R41 to R28, R45 to R29, R7 to R31, R52 to R310, R58 to R311, R64 to R312, R69 to R313, R74 to R314, R13 to R32, R18 to R33, R24 to R34, R29 to R35, R35 to R36, R39 to R37, R42 to R38, R46 to R39, R8 to R41, R53 to R410, R59 to R411, R65 to R412, R70 to R413, R75 to R414, R14 to R42, R19 to R43, R25 to R44, R30 to R45, R36 to R46, R40 to R47, R43 to R48, R47 to R49, R9 to R51, R54 to R510, R60 to R511, R66 to R512, R71 to R513, R76 to R514, R15 to R52, R20 to R53, R26 to R54, R31 to R55, R37 to R56, R48 to R59, R10 to R61, R55 to R610, R61 to R611, R77 to R614, R21 to R64, R32 to R66, R49 to R69
Connections:
- net labels added: 5VR, COL10, COL10R, COL11, COL12R, COL13, COL13R, COL7, COL7R, COL8, COL8R, COL9, COL9R, COl11R, COl12, LedGNDR, ROW0R, ROW1R, ROW2R, ROW3R, ROW4R, ROW5R
- wire segments 573 -> 488

Commit message: Finalized PCB and created Gerbers
Parts:
- removed M1: Mosfet-DMN63D8L, Ace's Footprints:Mosfet-DMN63D8L, symbol Ace's~Schematic~Symbols:Mosfet-DMN63D8L
- added M1: Mosfet-DMN63D8L, Aces Footprints:Mosfet-DMN63D8L, symbol Aces_Schematic_Symbols:Mosfet-DMN63D8L
- renumbered MXIL1 to MX_I1
Connections:
- net labels added: COL12
- net labels removed: COl12
- wire segments 488 -> 489
Changed lines of the file:
@@
 P 8875 3400
 AR Path="/5CE40BC3" Ref="MX?"  Part="1"
-AR Path="/5CDFA39B/5CE40BC3" Ref="MXIL1"  Part="1"
-F 0 "MXIL1" H 8961 3617 60  0000 C CNN
+AR Path="/5CDFA39B/5CE40BC3" Ref="MX_I1"  Part="1"
+F 0 "MX_I1" H 8961 3617 60  0000 C CNN
 F 1 "MX-1U" H 8961 3543 20  0000 C CNN
 F 2 "MX_Alps_Hybrid:MXOnly-1U" H 8850 3375 60  0001 C CNN
@@
 Wire Wire Line
 	4750 6075 5025 6075
-$Comp
-L Ace's~Schematic~Symbols:Mosfet-DMN63D8L M1
-U 1 1 5CA1B7FF
-P 5650 6075
-F 0 "M1" H 5827 6121 50  0000 L CNN
-F 1 "Mosfet-DMN63D8L" H 5827 6030 50  0000 L CNN
-F 2 "Ace's Footprints:Mosfet-DMN63D8L" H 5650 6075 50  0001 C CNN
-F 3 "" H 5650 6075 50  0001 C CNN
-	1    5650 6075
-	1    0    0    -1
-$EndComp
 Wire Wire Line
 	5650 6325 5650 6425
@@
 COL11
 Text GLabel 5375 4000 0    50   Input ~ 0
-COl12
+COL12
 Text GLabel 5375 3900 0    50   Input ~ 0
 COL13
@@
 Wire Wire Line
 	5005 3600 5375 3600
+Wire Wire Line
+	3800 3950 3800 3375
+Connection ~ 3800 3375
+$Comp
+L Aces_Schematic_Symbols:Mosfet-DMN63D8L M1
+U 1 1 5CA7C160
+P 5650 6075
+F 0 "M1" H 5827 6121 50  0000 L CNN
+F 1 "Mosfet-DMN63D8L" H 5827 6030 50  0000 L CNN
+F 2 "Aces Footprints:Mosfet-DMN63D8L" H 5650 6075 50  0001 C CNN
+F 3 "" H 5650 6075 50  0001 C CNN
+	1    5650 6075
+	1    0    0    -1
+$EndComp
 $EndSCHEMATC

Commit message: more pcb work
Parts:
- R11, R110, R111, R112, R113, R114, R12, R13, R14, R15, R16, R19, R21, R210, R211, R212, R213, R214, R22, R23, R24, R25, R26, R27, R28, R29, R31, R310, R311, R312, R313, R314, R32, R33, R34, R35, R36, R37, R38, R39, R41, R410, R411, R412, R413, R414, R42, R43, R44, R45, R46, R47, R48, R49, R51, R510, R511, R512, R513, R514, R52, R53, R54, R55, R56, R59, R61, R610, R611, R614, R64, R66, R69: value 800 -> 1k
